Commit message: World generator: several worlds, angled walls, and a body-clearance check
make_warehouse.py becomes make_worlds.py and describes each world as data.
Obstacles can now be turned (walls between any two points), which the
lettering needs.

It also gains a second check. The planner only keeps the lidar point 0.8 m
from obstacles, so it will happily route through a gap the robot's 1.4 m
body can't take. For every pair of areas, the generator compares the
planner's shortest route with one that stays 1.2 m clear, and rejects the
world if the planner's is more than 3 m shorter. On the first version of
the lettering it reports exactly the shortcut the robot crashed through.

The regenerated warehouse files only differ in their header comment and in
spelling out a zero rotation.

File: src/gazebo/launch/warehouse_env.urdf (robot description, URDF)
Before this commit: robot warehouse, 31 links, 30 joints
Joints:
- joint carton_0_joint: origin xyz=-13 10 2.75 -> xyz=-13 10 2.75 rpy=0 0 0
- joint carton_1_joint: origin xyz=-10.5 10 2.75 -> xyz=-10.5 10 2.75 rpy=0 0 0
- joint carton_2_joint: origin xyz=-8 10 2.75 -> xyz=-8 10 2.75 rpy=0 0 0
- joint carton_3_joint: origin xyz=-5.5 10 2.75 -> xyz=-5.5 10 2.75 rpy=0 0 0
- joint carton_4_joint: origin xyz=-3.5 10 2.75 -> xyz=-3.5 10 2.75 rpy=0 0 0
- joint crate_1_joint: origin xyz=3 -9 0.75 -> xyz=3 -9 0.75 rpy=0 0 0
- joint crate_2_joint: origin xyz=0.5 -12.5 0.75 -> xyz=0.5 -12.5 0.75 rpy=0 0 0
- joint desk_1_joint: origin xyz=-11.5 -10 0.65 -> xyz=-11.5 -10 0.65 rpy=0 0 0
- joint desk_2_joint: origin xyz=-6 -12 0.65 -> xyz=-6 -12 0.65 rpy=0 0 0
- joint lane_north_joint: origin xyz=0 3.9 0.005 -> xyz=0 3.9 0.005 rpy=0 0 0
- joint lane_south_joint: origin xyz=0 -3.9 0.005 -> xyz=0 -3.9 0.005 rpy=0 0 0
- joint pallets_1_joint: origin xyz=6.5 10 0.9 -> xyz=6.5 10 0.9 rpy=0 0 0
- joint pallets_2_joint: origin xyz=11.5 11.5 0.9 -> xyz=11.5 11.5 0.9 rpy=0 0 0
- joint pillar_1_joint: origin xyz=-2 1.8 1.5 -> xyz=-2 1.8 1.5 rpy=0 0 0
- joint pillar_2_joint: origin xyz=8 -1.8 1.5 -> xyz=8 -1.8 1.5 rpy=0 0 0
- joint rack_joint: origin xyz=-8.75 10 1.25 -> xyz=-8.75 10 1.25 rpy=0 0 0
- joint truck_joint: origin xyz=9.5 -12.2 1.6 -> xyz=9.5 -12.2 1.6 rpy=0 0 0
- joint wall_east_joint: origin xyz=15 0 1.5 -> xyz=15 0 1.5 rpy=0 0 0
- joint wall_hall_n1_joint: origin xyz=-12.5 5 1.5 -> xyz=-12.5 5 1.5 rpy=0 0 0
- joint wall_hall_n2_joint: origin xyz=0.5 5 1.5 -> xyz=0.5 5 1.5 rpy=0 0 0
- joint wall_hall_n3_joint: origin xyz=13 5 1.5 -> xyz=13 5 1.5 rpy=0 0 0
- joint wall_hall_s1_joint: origin xyz=-13 -5 1.5 -> xyz=-13 -5 1.5 rpy=0 0 0
- joint wall_hall_s2_joint: origin xyz=-1 -5 1.5 -> xyz=-1 -5 1.5 rpy=0 0 0
- joint wall_hall_s3_joint: origin xyz=12 -5 1.5 -> xyz=12 -5 1.5 rpy=0 0 0
- joint wall_north_joint: origin xyz=0 15 1.5 -> xyz=0 15 1.5 rpy=0 0 0
- joint wall_office_1_joint: origin xyz=-2 -13.5 1.5 -> xyz=-2 -13.5 1.5 rpy=0 0 0
- joint wall_office_2_joint: origin xyz=-2 -6 1.5 -> xyz=-2 -6 1.5 rpy=0 0 0
- joint wall_south_joint: origin xyz=0 -15 1.5 -> xyz=0 -15 1.5 rpy=0 0 0
- joint wall_storage_joint: origin xyz=2 7.6 1.5 -> xyz=2 7.6 1.5 rpy=0 0 0
- joint wall_west_joint: origin xyz=-15 0 1.5 -> xyz=-15 0 1.5 rpy=0 0 0
